Commit message: franka integration

File: providers/meca500/src/meca500_moveit/config/meca500.ros2_control.xacro (robot description, xacro)
@@ -8,5 +8,5 @@
          arg is declared in meca500.urdf.xacro and forwarded here. -->
     <xacro:arg name="simulation" default="false"/>
-    <xacro:macro name="meca500_ros2_control" params="name initial_positions_file robot_ip robot_port connect_timeout_ms response_timeout_ms">
+    <xacro:macro name="meca500_ros2_control" params="name initial_positions_file robot_ip robot_port connect_timeout_ms response_timeout_ms auto_home:=false">
         <xacro:property name="initial_positions" value="${load_yaml(initial_positions_file)['initial_positions']}"/>
         <ros2_control name="${name}" type="system">
@@ -29,4 +29,11 @@
                 <param name="connect_timeout_ms">${connect_timeout_ms}</param>
                 <param name="response_timeout_ms">${response_timeout_ms}</param>
+                <!-- Skip the activation-time Home command by default —
+                     Meca500 retains absolute encoder homing across power
+                     cycles, so once-per-power-on homing is sufficient and
+                     blocking the controller-manager activation on Home
+                     just slows MoveIt bringup. Pass auto_home:=true on
+                     `meca500-real-up` after a fresh power-on. -->
+                <param name="auto_home">${auto_home}</param>
             </hardware>
         </xacro:unless>

File: providers/meca500/src/meca500_moveit/config/meca500.urdf.xacro (robot description, xacro)
@@ -9,4 +9,9 @@
     <xacro:arg name="connect_timeout_ms" default="2000" />
     <xacro:arg name="response_timeout_ms" default="30000" />
+    <!-- Meca500 retains absolute joint encoders across power cycles, so
+         the activation-time Home command is unnecessary except after a
+         fresh power-on. Default off to keep MoveIt bringup snappy; flip
+         to "true" via the meca500_bringup launch arg of the same name. -->
+    <xacro:arg name="auto_home" default="false" />
     <!-- Seed-gripper overlay args. Defaults match meca500.xacro so leaving
          use_seed_gripper=false keeps the legacy Schunk geometry untouched.
@@ -49,4 +54,5 @@
         connect_timeout_ms="$(arg connect_timeout_ms)"
         response_timeout_ms="$(arg response_timeout_ms)"
+        auto_home="$(arg auto_home)"
     />
 </robot>
